File: PCB-NEW/rabbitholev1/rabbitholev1.kicad_pcb (KiCad board)
At the start: 2 copper layers, 314.6 x 105.4 mm, 149 parts, among them SW1 SW_Push, U1 ATmega32U4-AU, Y1 Crystal_GND24_Small

Commit message: d
Parts:
- moved R4 2.59 mm to (167.6, 127.6)
- moved R3 2.07 mm to (163.9, 128.0)
Routing:
- net D+: track 188.2 -> 185.7 mm
- net D-: track 191.0 -> 188.7 mm
- net Net-(D67-Pad2): track 37.0 -> 39.0 mm

Commit message: f
Parts:
- moved Y1 35.0 mm to (240.8, 188.6), turned to 45 degrees
- moved C2 31.4 mm to (227.1, 202.2), turned to 270 degrees
- moved C3 30.2 mm to (229.2, 202.2), turned to 270 degrees
- moved C4 28.8 mm to (231.3, 202.2), turned to 270 degrees
- moved C5 27.5 mm to (233.2, 202.2), turned to 270 degrees
- moved C6 26.5 mm to (235.3, 202.2)
- moved C7 26.5 mm to (237.4, 202.2)
- moved U1 25.5 mm to (250.7, 194.4), turned to 45 degrees
- moved R1 18.7 mm to (234.1, 206.4)
- moved C1 16.7 mm to (235.4, 198.5), turned to 270 degrees
- moved D67 16.4 mm to (154.4, 133.0)
- moved R2 14.8 mm to (237.4, 198.5), turned to 270 degrees
- moved SW1 10.1 mm to (243.5, 208.0)
- moved 500m1 2.95 mm to (148.8, 128.8)
Connections:
- MX65 pad 1: col12 -> col13
- MX66 pad 1: col12 -> col14
- U1 pad 1: row0 -> row4
- U1 pad 19: col2 -> col10
- U1 pad 20: col1 -> col12
- U1 pad 21: col0 -> col9
- U1 pad 22: col3 -> col8
- U1 pad 25: col4 -> col7
- U1 pad 26: col5 -> col6
- U1 pad 27: col6 -> col5
- U1 pad 28: col7 -> col4
- U1 pad 29: col8 -> col13
- U1 pad 30: col9 -> col14
- U1 pad 31: col10 -> col3
- U1 pad 32: col11 -> col2
- U1 pad 36: col12 -> col1
- U1 pad 37: col13 -> col0
- U1 pad 38: row2 -> row1
- U1 pad 39: row4 -> row2
- U1 pad 40: row3 -> row0
- U1 pad 41: row1 -> row3
- U1 pad 8: col14 -> col11
Routing:
- net col0: track 320.8 -> 455.1 mm
- net col1: track 304.3 -> 436.3 mm
- net col2: track 282.5 -> 411.4 mm
- net col12: track 214.7 -> 100.5 mm
- net col3: track 256.8 -> 369.5 mm, vias 1 -> 0
- net col6: track 198.9 -> 254.7 mm, vias 1 -> 0
- net D+: track 185.7 -> 238.8 mm, vias 4 -> 2
- net col9: track 125.2 -> 176.6 mm, vias 1 -> 0
- net D-: track 188.7 -> 237.9 mm, vias 4 -> 2
- net col14: track 181.5 -> 133.2 mm, vias 7 -> 1
- net col5: track 209.8 -> 255.7 mm, vias 1 -> 0
- net col13: track 161.8 -> 116.5 mm, vias 3 -> 0
- net col8: track 150.8 -> 195.9 mm, vias 1 -> 0
- net col4: track 229.4 -> 274.1 mm, vias 1 -> 0
- net col7: track 170.3 -> 212.8 mm, vias 1 -> 0
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